File: hardware/rearbox/brake_light.kicad_sch (KiCad schematic)
At the start: 8 parts, among them Q1 BUK6D210, Q2 BUK6D210

Commit message: Functional new CAN library and fixed SDC sensing problems
Other:
- company: Author: I. Kajdan -> Author: J. Kasprzyk
