File: hardware/rearbox/can_transceiver.kicad_sch (KiCad schematic)
At the start: 15 parts, among them U7 ADM3057ExRW

Commit message: Functional new CAN library and fixed SDC sensing problems
Other:
- company: Author: I. Kajdan -> Author: J. Kasprzyk
