File: hardware/rearbox/rearbox.kicad_sch (KiCad schematic)
At the start: 25 parts, among them J1 STDC14, J2 ST-LINK, J5 XIAO ESP32S3 Sense, U1 LM4040C33FTA, U2 STM32G473RCTx, Y1 48MHz

Commit message: Functional new CAN library and fixed SDC sensing problems
Other:
- company: Author: I. Kajdan -> Author: J. Kasprzyk
