File: hardware/rearbox/safety_input.kicad_sch (KiCad schematic)
At the start: 9 parts, among them U10 TLP291-4

Commit message: Functional new CAN library and fixed SDC sensing problems
Other:
- company: Author: I. Kajdan -> Author: J. Kasprzyk
