File: hardware/rearbox/safety_inputs.kicad_sch (KiCad schematic)
At the start: 9 parts, among them U9 TCA6416ARTWR

Commit message: Functional new CAN library and fixed SDC sensing problems
Other:
- company: Author: I. Kajdan -> Author: J. Kasprzyk
